File: hardware/picovic.sch (KiCad schematic (older format))
At the start: 13 parts, among them J1 Mini-DIN-6, J2 DB15_Female_HighDensity, U1 Pico, U2 SN74LVC4245A

Commit message: update schematic
Parts:
- R2, R5: value R_Small -> 1k
- R3, R6, R8: value R_Small -> 500R
- R4, R7, R9: value R_Small -> 250R
Connections:
- net GND: now also U1.13 (GND), U1.18 (GND), U1.23 (GND), U1.28 (GND), U1.3 (GND), U1.33 (AGND), U1.38 (GND), U1.42 (GND), U1.8 (GND)
Changed lines of the file:
@@
 P 8200 2100
 F 0 "R3" V 8004 2100 50  0000 C CNN
-F 1 "R_Small" V 8095 2100 50  0000 C CNN
+F 1 "500R" V 8095 2100 50  0000 C CNN
 F 2 "Resistor_THT:R_Axial_DIN0204_L3.6mm_D1.6mm_P7.62mm_Horizontal" H 8200 2100 50  0001 C CNN
 F 3 "~" H 8200 2100 50  0001 C CNN
@@
 P 8200 2300
 F 0 "R4" V 8004 2300 50  0000 C CNN
-F 1 "R_Small" V 8095 2300 50  0000 C CNN
+F 1 "250R" V 8095 2300 50  0000 C CNN
 F 2 "Resistor_THT:R_Axial_DIN0204_L3.6mm_D1.6mm_P7.62mm_Horizontal" H 8200 2300 50  0001 C CNN
 F 3 "~" H 8200 2300 50  0001 C CNN
@@
 P 8200 2500
 F 0 "R5" V 8004 2500 50  0000 C CNN
-F 1 "R_Small" V 8095 2500 50  0000 C CNN
+F 1 "1k" V 8095 2500 50  0000 C CNN
 F 2 "Resistor_THT:R_Axial_DIN0204_L3.6mm_D1.6mm_P7.62mm_Horizontal" H 8200 2500 50  0001 C CNN
 F 3 "~" H 8200 2500 50  0001 C CNN
@@
 P 8200 2700
 F 0 "R6" V 8004 2700 50  0000 C CNN
-F 1 "R_Small" V 8095 2700 50  0000 C CNN
+F 1 "500R" V 8095 2700 50  0000 C CNN
 F 2 "Resistor_THT:R_Axial_DIN0204_L3.6mm_D1.6mm_P7.62mm_Horizontal" H 8200 2700 50  0001 C CNN
 F 3 "~" H 8200 2700 50  0001 C CNN
@@
 P 8200 2900
 F 0 "R7" V 8004 2900 50  0000 C CNN
-F 1 "R_Small" V 8095 2900 50  0000 C CNN
+F 1 "250R" V 8095 2900 50  0000 C CNN
 F 2 "Resistor_THT:R_Axial_DIN0204_L3.6mm_D1.6mm_P7.62mm_Horizontal" H 8200 2900 50  0001 C CNN
 F 3 "~" H 8200 2900 50  0001 C CNN
@@
 P 8200 3100
 F 0 "R8" V 8004 3100 50  0000 C CNN
-F 1 "R_Small" V 8095 3100 50  0000 C CNN
+F 1 "500R" V 8095 3100 50  0000 C CNN
 F 2 "Resistor_THT:R_Axial_DIN0204_L3.6mm_D1.6mm_P7.62mm_Horizontal" H 8200 3100 50  0001 C CNN
 F 3 "~" H 8200 3100 50  0001 C CNN
@@
 P 8200 1900
 F 0 "R2" V 8004 1900 50  0000 C CNN
-F 1 "R_Small" V 8095 1900 50  0000 C CNN
+F 1 "1k" V 8095 1900 50  0000 C CNN
 F 2 "Resistor_THT:R_Axial_DIN0204_L3.6mm_D1.6mm_P7.62mm_Horizontal" H 8200 1900 50  0001 C CNN
 F 3 "~" H 8200 1900 50  0001 C CNN
@@
 P 8200 3300
 F 0 "R9" V 8004 3300 50  0000 C CNN
-F 1 "R_Small" V 8095 3300 50  0000 C CNN
+F 1 "250R" V 8095 3300 50  0000 C CNN
 F 2 "Resistor_THT:R_Axial_DIN0204_L3.6mm_D1.6mm_P7.62mm_Horizontal" H 8200 3300 50  0001 C CNN
 F 3 "~" H 8200 3300 50  0001 C CNN
@@
 Wire Wire Line
 	4250 3950 4850 3950
+$Comp
+L power:GND #PWR?
+U 1 1 61168BA1
+P 5550 4950
+F 0 "#PWR?" H 5550 4700 50  0001 C CNN
+F 1 "GND" H 5555 4777 50  0000 C CNN
+F 2 "" H 5550 4950 50  0001 C CNN
+F 3 "" H 5550 4950 50  0001 C CNN
+	1    5550 4950
+	-1   0    0    -1
+$EndComp
+$Comp
+L power:GND #PWR?
+U 1 1 6116C3D3
+P 4650 4550
+F 0 "#PWR?" H 4650 4300 50  0001 C CNN
+F 1 "GND" H 4655 4377 50  0000 C CNN
+F 2 "" H 4650 4550 50  0001 C CNN
+F 3 "" H 4650 4550 50  0001 C CNN
+	1    4650 4550
+	-1   0    0    -1
+$EndComp
+Wire Wire Line
+	4850 4550 4650 4550
+$Comp
+L power:GND #PWR?
+U 1 1 611735AD
+P 4650 4050
+F 0 "#PWR?" H 4650 3800 50  0001 C CNN
+F 1 "GND" H 4655 3877 50  0000 C CNN
+F 2 "" H 4650 4050 50  0001 C CNN
+F 3 "" H 4650 4050 50  0001 C CNN
+	1    4650 4050
+	-1   0    0    -1
+$EndComp
+Wire Wire Line
+	4850 4050 4650 4050
+$Comp
+L power:GND #PWR?
+U 1 1 6117AD86
+P 4650 3550
+F 0 "#PWR?" H 4650 3300 50  0001 C CNN
+F 1 "GND" H 4655 3377 50  0000 C CNN
+F 2 "" H 4650 3550 50  0001 C CNN
+F 3 "" H 4650 3550 50  0001 C CNN
+	1    4650 3550
+	-1   0    0    -1
+$EndComp
+Wire Wire Line
+	4850 3550 4650 3550
+$Comp
+L power:GND #PWR?
+U 1 1 611829B8
+P 4700 3050
+F 0 "#PWR?" H 4700 2800 50  0001 C CNN
+F 1 "GND" H 4705 2877 50  0000 C CNN
+F 2 "" H 4700 3050 50  0001 C CNN
+F 3 "" H 4700 3050 50  0001 C CNN
+	1    4700 3050
+	-1   0    0    -1
+$EndComp
+Wire Wire Line
+	4850 3050 4700 3050
+$Comp
+L power:GND #PWR?
+U 1 1 6118A571
+P 6400 3050
+F 0 "#PWR?" H 6400 2800 50  0001 C CNN
+F 1 "GND" H 6405 2877 50  0000 C CNN
+F 2 "" H 6400 3050 50  0001 C CNN
+F 3 "" H 6400 3050 50  0001 C CNN
+	1    6400 3050
+	-1   0    0    -1
+$EndComp
+Wire Wire Line
+	6400 3050 6250 3050
+$Comp
+L power:GND #PWR?
+U 1 1 611922EA
+P 6400 3550
+F 0 "#PWR?" H 6400 3300 50  0001 C CNN
+F 1 "GND" H 6405 3377 50  0000 C CNN
+F 2 "" H 6400 3550 50  0001 C CNN
+F 3 "" H 6400 3550 50  0001 C CNN
+	1    6400 3550
+	-1   0    0    -1
+$EndComp
+Wire Wire Line
+	6400 3550 6250 3550
+$Comp
+L power:GND #PWR?
+U 1 1 6119A50C
+P 6450 4050
+F 0 "#PWR?" H 6450 3800 50  0001 C CNN
+F 1 "GND" H 6455 3877 50  0000 C CNN
+F 2 "" H 6450 4050 50  0001 C CNN
+F 3 "" H 6450 4050 50  0001 C CNN
+	1    6450 4050
+	-1   0    0    -1
+$EndComp
+Wire Wire Line
+	6450 4050 6250 4050
+$Comp
+L power:GND #PWR?
+U 1 1 611A2922
+P 6450 4550
+F 0 "#PWR?" H 6450 4300 50  0001 C CNN
+F 1 "GND" H 6455 4377 50  0000 C CNN
+F 2 "" H 6450 4550 50  0001 C CNN
+F 3 "" H 6450 4550 50  0001 C CNN
+	1    6450 4550
+	-1   0    0    -1
+$EndComp
+Wire Wire Line
+	6450 4550 6250 4550
 $EndSCHEMATC
