File: hardware/picovic.kicad_pcb (KiCad board)
At the start: 2 copper layers, 54.6 x 53.3 mm, 16 parts, among them J1 DB15_Female_HighDensity, J2 Conn_01x06, P1 Mini-DIN_6pins_ver2, U1 74HC14

Commit message: Fix violations
Parts:
- added C1: 0.1uF, Capacitor_THT:C_Disc_D5.0mm_W2.5mm_P5.00mm, F.Cu at (60.7, 12.7)
- added C2: 0.1uF, Capacitor_THT:C_Disc_D5.0mm_W2.5mm_P5.00mm, F.Cu at (60.7, 16.0)
- moved REF** 29.8 mm to (36.7, 24.5)
Routing:
- net +5V: track 83.6 -> 89.1 mm
- net +3.3V: track 64.9 -> 68.4 mm
- net Net-(J1-Pad3): track 20.8 -> 21.7 mm
